Commit message: add cameras in xacro for demo 5 and 6

File: agimus_demo_05_pick_and_place/urdf/demo.urdf.xacro (robot description, xacro)
@@ -1,7 +1,6 @@
 <?xml version='1.0' encoding='utf-8'?>
 <robot xmlns:xacro="http://www.ros.org/wiki/xacro" name="panda">
-  <xacro:include filename="$(find franka_description)/robots/fer/fer.urdf.xacro">
-    <!-- <xacro:arg name="with_sc" value="True" /> -->
-  </xacro:include>
+  <xacro:arg name="use_camera" default="true" />
+  <xacro:include filename="$(find franka_description)/robots/fer/fer.urdf.xacro"/>
   <xacro:include filename="$(find agimus_demo_05_pick_and_place)/urdf/support.urdf.xacro"/>
   <xacro:support/>
@@ -9,4 +8,4 @@
     <parent link="robot_attachment_link" />
     <child link="base" />
-</joint>
+  </joint>
 </robot>

File: agimus_demo_06_regrasp/urdf/demo.urdf.xacro (robot description, xacro)
@@ -1,7 +1,6 @@
 <?xml version='1.0' encoding='utf-8'?>
 <robot xmlns:xacro="http://www.ros.org/wiki/xacro" name="panda">
-  <xacro:include filename="$(find franka_description)/robots/fer/fer.urdf.xacro">
-    <!-- <xacro:arg name="with_sc" value="True" /> -->
-  </xacro:include>
+  <xacro:arg name="use_camera" default="true" />
+  <xacro:include filename="$(find franka_description)/robots/fer/fer.urdf.xacro"/>
   <xacro:include filename="$(find agimus_demo_06_regrasp)/urdf/support.urdf.xacro"/>
   <xacro:support/>
@@ -9,4 +8,4 @@
     <parent link="robot_attachment_link" />
     <child link="base" />
-</joint>
+  </joint>
 </robot>

Commit message: Still need to make robot model harmonized between ros and hpp

File: agimus_demo_05_pick_and_place/urdf/demo.urdf.xacro (robot description, xacro)
@@ -6,4 +6,9 @@
   <xacro:arg name="ee_id" default="franka_hand_with_camera"/>
   <xacro:arg name="use_camera" default="true"/>
+  <xacro:property name="arm_id" value="$(arg arm_id)" />
+  <xacro:property name="ee_id" value="$(arg ee_id)" />
+  <xacro:property name="use_camera" value="$(arg use_camera)" />
+  <xacro:property name="hand" value="$(arg hand)" />
+  <xacro:property name="with_sc" value="$(arg with_sc)" />
   <xacro:include filename="$(find franka_description)/robots/${arm_id}/${arm_id}.urdf.xacro"/>
   <xacro:include filename="$(find agimus_demo_05_pick_and_place)/urdf/support.urdf.xacro"/>
