Commit message: Settings that makes the robot a bit off wrt the target

File: agimus_demo_05_pick_and_place/urdf/big_box.urdf (robot description, URDF)
Before this commit: robot big_box, 1 links, 0 joints
Links:
- link base_link: geometry collision box size=0.0 0.0 0.0; collision box size=0.0 0.0 0.0

File: agimus_demo_05_pick_and_place/urdf/robot_with_camera.urdf.xacro (robot description, xacro)
@@ -257,5 +257,4 @@
   <link name="fer_hand">
     <visual name="fer_hand_visual">
-      <origin rpy="0 0 -0.7853981633974483" xyz="0 0 0"/>
       <geometry>
         <mesh filename="package://franka_description/meshes/robot_ee/franka_hand_white/visual/hand.dae"/>
@@ -263,5 +262,4 @@
     </visual>
     <collision name="fer_hand_collision">
-      <origin rpy="0 0 -0.7853981633974483" xyz="0 0 0"/>
       <geometry>
         <mesh filename="package://franka_description/meshes/robot_ee/franka_hand_white/collision/hand.stl"/>
@@ -283,5 +281,4 @@
   <link name="fer_leftfinger">
     <visual name="fer_leftfinger_visual">
-      <origin rpy="0 0 -0.7853981633974483" xyz="0 0 0"/>
       <geometry>
         <mesh filename="package://franka_description/meshes/robot_ee/franka_hand_white/visual/finger.dae"/>
@@ -319,5 +316,5 @@
   <link name="fer_rightfinger">
     <visual name="fer_rightfinger_visual">
-      <origin rpy="0 0 2.356194490192345" xyz="0 0 0"/>
+      <origin rpy="0 0 3.141592653589793" xyz="0 0 0"/>
       <geometry>
         <mesh filename="package://franka_description/meshes/robot_ee/franka_hand_white/visual/finger.dae"/>
@@ -374,5 +371,5 @@
     <parent link="fer_link8"/>
     <child link="fer_ref_camera_link"/>
-    <origin rpy="1.05427421                       -1.56738918                       1.26092726" xyz="0.02506404                       -0.02921068                       0.02847444"/>
+    <origin rpy="1.05427421  -1.56738918  1.26092726" xyz="0.02506404 -0.02921068 0.02847444"/>
   </joint>
   <material name="aluminum">
@@ -456,5 +453,5 @@
   <!-- camera color joints and links -->
   <joint name="camera_color_joint" type="fixed">
-    <origin rpy="0 0 0" xyz="0 0.015 0"/>
+    <origin rpy="-0.010 0.006 -0.003" xyz="0 0.015 0"/>
     <parent link="camera_link"/>
     <child link="camera_color_frame"/>

File: agimus_demo_05_pick_and_place/urdf/support.urdf.xacro (robot description, xacro)
@@ -200,5 +200,5 @@
     <link name="robot_attachment_link" />
     <joint name="support_joint" type="fixed">
-      <origin xyz="0.422 0.0 .92" rpy="0 0 ${pi}" />
+      <origin xyz="0.422 0.0 .90" rpy="0 0 ${pi}" />
       <parent link="support_link" />
       <child link="robot_attachment_link" />

Commit message: changes from Kat for demo

File: agimus_demo_05_pick_and_place/urdf/big_box.urdf (robot description, URDF)
Before this commit: robot big_box, 1 links, 0 joints
Links:
- link base_link: geometry collision box size=0.001 0.367 0.22; collision box size=0.001 0.367 0.22
