Commit message: update demo 08 for cosmik compatibility

File: agimus_demo_08_collision_avoidance/urdf/environment.urdf.xacro (robot description, xacro)
@@ -3,4 +3,7 @@
   <material name="blue">
     <color rgba="0.1 0.1 0.8 0.5"/>
+  </material>
+  <material name="human_obstacle">
+    <color rgba="0.1 0.6 1.0 0.6"/>
   </material>
   <link name="obstacle">
@@ -22,3 +25,28 @@
     </inertial>
   </link>
+  <!-- Dynamic RT-COSMIK obstacles visualized from TF frames obstacle_0/1/2. -->
+  <link name="obstacle_0">
+    <visual>
+      <geometry>
+        <cylinder radius="0.045" length="0.22"/>
+      </geometry>
+      <material name="human_obstacle"/>
+    </visual>
+  </link>
+  <link name="obstacle_1">
+    <visual>
+      <geometry>
+        <cylinder radius="0.035" length="0.20"/>
+      </geometry>
+      <material name="human_obstacle"/>
+    </visual>
+  </link>
+  <link name="obstacle_2">
+    <visual>
+      <geometry>
+        <cylinder radius="0.03" length="0.12"/>
+      </geometry>
+      <material name="human_obstacle"/>
+    </visual>
+  </link>
 </robot>

Commit message: avoids two root link in env xacro

File: agimus_demo_08_collision_avoidance/urdf/environment.urdf.xacro (robot description, xacro)
@@ -1,4 +1,8 @@
 <?xml version="1.0"?>
 <robot xmlns:xacro="http://www.ros.org/wiki/xacro" name="obstacle">
+  <xacro:arg name="use_rtcosmik_obstacles" default="false"/>
+  <xacro:property
+    name="use_rtcosmik_obstacles"
+    value="$(arg use_rtcosmik_obstacles)"/>
   <material name="blue">
     <color rgba="0.1 0.1 0.8 0.5"/>
@@ -7,46 +11,82 @@
     <color rgba="0.1 0.6 1.0 0.6"/>
   </material>
-  <link name="obstacle">
-    <visual>
-      <geometry>
-        <sphere radius="0.1"/>
-      </geometry>
-      <material name="blue"/>
-    </visual>
-    <collision>
-      <geometry>
-        <sphere radius="0.1"/>
-      </geometry>
-    </collision>
-    <inertial>
-      <origin rpy="0 0 0" xyz="0 0 0"/>
-      <mass value="10.0"/>
-      <inertia ixx="1.67" ixy="0" ixz="0" iyy="1.67" iyz="0" izz="1.67"/>
-    </inertial>
-  </link>
-  <!-- Dynamic RT-COSMIK obstacles visualized from TF frames obstacle_0/1/2. -->
-  <link name="obstacle_0">
-    <visual>
-      <geometry>
-        <cylinder radius="0.045" length="0.22"/>
-      </geometry>
-      <material name="human_obstacle"/>
-    </visual>
-  </link>
-  <link name="obstacle_1">
-    <visual>
-      <geometry>
-        <cylinder radius="0.035" length="0.20"/>
-      </geometry>
-      <material name="human_obstacle"/>
-    </visual>
-  </link>
-  <link name="obstacle_2">
-    <visual>
-      <geometry>
-        <cylinder radius="0.03" length="0.12"/>
-      </geometry>
-      <material name="human_obstacle"/>
-    </visual>
-  </link>
+  <xacro:unless value="${use_rtcosmik_obstacles == 'true'}">
+    <link name="obstacle">
+      <visual>
+        <geometry>
+          <sphere radius="0.1"/>
+        </geometry>
+        <material name="blue"/>
+      </visual>
+      <collision name="obstacle_0">
+        <geometry>
+          <sphere radius="0.1"/>
+        </geometry>
+      </collision>
+      <inertial>
+        <origin rpy="0 0 0" xyz="0 0 0"/>
+        <mass value="10.0"/>
+        <inertia ixx="1.67" ixy="0" ixz="0" iyy="1.67" iyz="0" izz="1.67"/>
+      </inertial>
+    </link>
+  </xacro:unless>
+  <xacro:if value="${use_rtcosmik_obstacles == 'true'}">
+    <link name="obstacle_root"/>
+    <!-- Dynamic RT-COSMIK obstacles. -->
+    <link name="obstacle_0">
+      <visual>
+        <geometry>
+          <cylinder radius="0.045" length="0.22"/>
+        </geometry>
+        <material name="human_obstacle"/>
+      </visual>
+      <collision name="obstacle_0">
+        <geometry>
+          <cylinder radius="0.045" length="0.22"/>
+        </geometry>
+      </collision>
+    </link>
+    <link name="obstacle_1">
+      <visual>
+        <geometry>
+          <cylinder radius="0.035" length="0.20"/>
+        </geometry>
+        <material name="human_obstacle"/>
+      </visual>
+      <collision name="obstacle_1">
+        <geometry>
+          <cylinder radius="0.035" length="0.20"/>
+        </geometry>
+      </collision>
+    </link>
+    <link name="obstacle_2">
+      <visual>
+        <geometry>
+          <cylinder radius="0.03" length="0.12"/>
+        </geometry>
+        <material name="human_obstacle"/>
+      </visual>
+      <collision name="obstacle_2">
+        <geometry>
+          <cylinder radius="0.03" length="0.12"/>
+        </geometry>
+      </collision>
+    </link>
+    <!-- Keep one rooted kinematic tree for robot_state_publisher. -->
+    <joint name="obstacle_root_to_obstacle_0" type="fixed">
+      <parent link="obstacle_root"/>
+      <child link="obstacle_0"/>
+      <origin xyz="0 0 0" rpy="0 0 0"/>
+    </joint>
+    <joint name="obstacle_root_to_obstacle_1" type="fixed">
+      <parent link="obstacle_root"/>
+      <child link="obstacle_1"/>
+      <origin xyz="0 0 0" rpy="0 0 0"/>
+    </joint>
+    <joint name="obstacle_root_to_obstacle_2" type="fixed">
+      <parent link="obstacle_root"/>
+      <child link="obstacle_2"/>
+      <origin xyz="0 0 0" rpy="0 0 0"/>
+    </joint>
+  </xacro:if>
 </robot>

Commit message: fix xacro tree

File: agimus_demo_08_collision_avoidance/urdf/environment.urdf.xacro (robot description, xacro)
@@ -2,7 +2,4 @@
 <robot xmlns:xacro="http://www.ros.org/wiki/xacro" name="obstacle">
   <xacro:arg name="use_rtcosmik_obstacles" default="false"/>
-  <xacro:property
-    name="use_rtcosmik_obstacles"
-    value="$(arg use_rtcosmik_obstacles)"/>
   <material name="blue">
     <color rgba="0.1 0.1 0.8 0.5"/>
@@ -11,5 +8,5 @@
     <color rgba="0.1 0.6 1.0 0.6"/>
   </material>
-  <xacro:unless value="${use_rtcosmik_obstacles == 'true'}">
+  <xacro:unless value="$(arg use_rtcosmik_obstacles)">
     <link name="obstacle">
       <visual>
@@ -31,5 +28,5 @@
     </link>
   </xacro:unless>
-  <xacro:if value="${use_rtcosmik_obstacles == 'true'}">
+  <xacro:if value="$(arg use_rtcosmik_obstacles)">
     <link name="obstacle_root"/>
     <!-- Dynamic RT-COSMIK obstacles. -->

Commit message: new tries ?

File: agimus_demo_08_collision_avoidance/urdf/environment.urdf.xacro (robot description, xacro)
@@ -38,5 +38,5 @@
         <material name="human_obstacle"/>
       </visual>
-      <collision name="obstacle_0">
+      <collision name="obstacle_0_0">
         <geometry>
           <cylinder radius="0.045" length="0.22"/>
@@ -51,5 +51,5 @@
         <material name="human_obstacle"/>
       </visual>
-      <collision name="obstacle_1">
+      <collision name="obstacle_1_0">
         <geometry>
           <cylinder radius="0.035" length="0.20"/>
@@ -64,5 +64,5 @@
         <material name="human_obstacle"/>
       </visual>
-      <collision name="obstacle_2">
+      <collision name="obstacle_2_0">
         <geometry>
           <cylinder radius="0.03" length="0.12"/>
